File: kicad/spigate.kicad_pcb (KiCad board)
At the start: 4 copper layers, 99.7 x 52.7 mm, 30 parts, among them J1 Conn_01x09, J2 n8 Bus Connector, J5 SD_CARD_PORT, U1 74LS393, U10 74LS153, U11 74HC273, U12 74HC245, U2 74HC00, U3 74LS139, U4 74HC04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

Commit message: shipped board
Changed lines of the file:
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@@
 		(tags "THT DIP DIL PDIP 2.54mm 7.62mm 300mil Socket")
 		(property "Reference" "U12"
-			(at 3.81 11.425 90)
+			(at 3.81 7.7928 90)
 			(layer "F.SilkS")
 			(effects
@@
 		(tags "THT DIP DIL PDIP 2.54mm 7.62mm 300mil Socket")
 		(property "Reference" "U11"
-			(at 3.76936 11.3742 90)
-			(layer "F.SilkS")
-			(effects
+			(at 3.74396 7.5642 90)
+			(layer "F.SilkS")
+			(effects
