File: kicad/spigate.kicad_sch (KiCad schematic)
At the start: 30 parts, among them J1 Conn_01x09, J2 n8 Bus Connector, J5 SD_CARD_PORT, U1 74LS393, U10 74LS153, U11 74HC273, U12 74HC245, U2 74HC00, U3 74LS139, U4 74HC04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

Commit message: shipped board
Connections:
- net +5V: now also U9.10 (~{S}); no longer U9.11 (C)
- net ~{DATA_WR}: now also U9.11 (C); no longer U9.10 (~{S})
Other:
- moved on the sheet: D1, R1
Changed lines of the file:
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@@
 	)
 	(junction
-		(at 97.79 208.28)
-		(diameter 0)
-		(color 0 0 0 0)
-	)
-	(junction
 		(at 292.1 200.66)
 		(diameter 0)
@@
 	)
 	(junction
+		(at 121.92 208.28)
+		(diameter 0)
+		(color 0 0 0 0)
+	)
+	(junction
 		(at 330.2 200.66)
 		(diameter 0)
@@
 	)
 	(junction
-		(at 120.65 208.28)
-		(diameter 0)
-		(color 0 0 0 0)
-	)
-	(junction
 		(at 78.74 77.47)
 		(diameter 0)
@@
 	(wire
 		(pts
+			(xy 121.92 208.28) (xy 123.19 208.28)
+		)
+		(stroke
+			(width 0)
+			(type default)
+		)
+	)
+	(wire
+		(pts
 			(xy 327.66 238.76) (xy 340.36 238.76)
 		)
@@
 	(wire
 		(pts
-			(xy 120.65 208.28) (xy 120.65 223.52)
+			(xy 121.92 208.28) (xy 121.92 223.52)
 		)
 		(stroke
@@
 	(wire
 		(pts
-			(xy 107.95 201.93) (xy 107.95 203.2)
-		)
-		(stroke
-			(width 0)
-			(type default)
-		)
-	)
-	(wire
-		(pts
-			(xy 115.57 208.28) (xy 120.65 208.28)
+			(xy 115.57 208.28) (xy 121.92 208.28)
 		)
 		(stroke
@@
 	(wire
 		(pts
-			(xy 85.09 223.52) (xy 120.65 223.52)
+			(xy 85.09 223.52) (xy 121.92 223.52)
 		)
 		(stroke
@@
 	(wire
 		(pts
-			(xy 116.84 207.01) (xy 116.84 213.36)
+			(xy 118.11 207.01) (xy 118.11 213.36)
 		)
 		(stroke
@@
 	(wire
 		(pts
-			(xy 120.65 208.28) (xy 123.19 208.28)
-		)
-		(stroke
-			(width 0)
-			(type default)
-		)
-	)
-	(wire
-		(pts
 			(xy 314.96 234.95) (xy 314.96 238.76)
 		)
@@
 	(wire
 		(pts
+			(xy 107.95 200.66) (xy 107.95 203.2)
+		)
+		(stroke
+			(width 0)
+			(type default)
+		)
+	)
+	(wire
+		(pts
 			(xy 85.09 223.52) (xy 85.09 255.27)
 		)
@@
 	(wire
 		(pts
-			(xy 100.33 210.82) (xy 97.79 210.82)
-		)
-		(stroke
-			(width 0)
-			(type default)
-		)
-	)
-	(wire
-		(pts
 			(xy 215.9 264.16) (xy 215.9 261.62)
 		)
@@
 	(wire
 		(pts
-			(xy 116.84 191.77) (xy 116.84 193.04)
+			(xy 118.11 191.77) (xy 118.11 193.04)
 		)
 		(stroke
@@
 	(wire
 		(pts
-			(xy 116.84 198.12) (xy 116.84 199.39)
+			(xy 118.11 198.12) (xy 118.11 199.39)
 		)
 		(stroke
@@
 	(wire
 		(pts
-			(xy 102.87 201.93) (xy 107.95 201.93)
-		)
-		(stroke
-			(width 0)
-			(type default)
-		)
-	)
-	(wire
-		(pts
 			(xy 91.44 52.07) (xy 92.71 52.07)
 		)
@@
 	(wire
 		(pts
-			(xy 116.84 213.36) (xy 115.57 213.36)
+			(xy 118.11 213.36) (xy 115.57 213.36)
 		)
 		(stroke
@@
 		)
 	)
-	(wire
-		(pts
-			(xy 97.79 210.82) (xy 97.79 208.28)
-		)
-		(stroke
-			(width 0)
-			(type default)
-		)
-	)
 	(polyline
 		(pts
@@
 	(wire
 		(pts
+			(xy 97.79 210.82) (xy 100.33 210.82)
+		)
+		(stroke
+			(width 0)
+			(type default)
+		)
+	)
+	(wire
+		(pts
 			(xy 123.19 146.05) (xy 125.73 146.05)
 		)
@@
 		)
 	)
-	(global_label "~{DATA_WR}"
-		(shape input)
-		(at 102.87 201.93 180)
-		(fields_autoplaced yes)
-		(effects
-			(font
-				(size 1.27 1.27)
-			)
-			(justify right)
-		)
-		(property "Intersheetrefs" "${INTERSHEET_REFS}"
-			(at -5.715 4.445 0)
-			(effects
-				(font
-					(size 1.27 1.27)
-				)
-				(hide yes)
-			)
-		)
-	)
 	(global_label "~{CS0}"
 		(shape input)
@@
 		)
 	)
+	(global_label "~{DATA_WR}"
+		(shape input)
+		(at 97.79 210.82 180)
+		(fields_autoplaced yes)
+		(effects
+			(font
+				(size 1.27 1.27)
+			)
+			(justify right)
+		)
+		(property "Intersheetrefs" "${INTERSHEET_REFS}"
+			(at -10.795 13.335 0)
+			(effects
+				(font
+					(size 1.27 1.27)
+				)
+				(hide yes)
+			)
+		)
+	)
 	(global_label "~{CTRL_WR}"
 		(shape input)
@@
 		(dnp no)
 		(property "Reference" "U9"
-			(at 107.95 198.6026 0)
+			(at 110.49 201.93 0)
 			(effects
 				(font
@@
 		)
 		(property "Value" "74HC74"
-			(at 107.95 200.914 0)
+			(at 112.522 203.962 0)
 			(effects
 				(font
@@
 	(symbol
 		(lib_id "Device:R_Small")
-		(at 116.84 195.58 0)
+		(at 118.11 195.58 0)
 		(unit 1)
 		(exclude_from_sim no)
@@
 		(fields_autoplaced yes)
 		(property "Reference" "R1"
-			(at 119.38 194.3099 0)
+			(at 120.65 194.3099 0)
 			(effects
 				(font
@@
 		)
 		(property "Value" "330R"
-			(at 119.38 196.8499 0)
+			(at 120.65 196.8499 0)
 			(effects
 				(font
@@
 		)
 		(property "Footprint" "Resistor_SMD:R_0805_2012Metric_Pad1.20x1.40mm_HandSolder"
-			(at 116.84 195.58 0)
+			(at 118.11 195.58 0)
 			(effects
 				(font
@@
 		)
 		(property "Datasheet" "~"
-			(at 116.84 195.58 0)
+			(at 118.11 195.58 0)
 			(effects
 				(font
@@
 		)
 		(property "Description" "Resistor, small symbol"
-			(at 116.84 195.58 0)
+			(at 118.11 195.58 0)
 			(effects
 				(font
@@
 	)
 	(symbol
+		(lib_id "power:+5V")
+		(at 107.95 200.66 0)
+		(unit 1)
+		(exclude_from_sim no)
+		(in_bom yes)
+		(on_board yes)
+		(dnp no)
+		(property "Reference" "#PWR08"
+			(at 107.95 204.47 0)
+			(effects
+				(font
+					(size 1.27 1.27)
+				)
+				(hide yes)
+			)
+		)
+		(property "Value" "+5V"
+			(at 104.394 199.898 0)
+			(effects
+				(font
+					(size 1.27 1.27)
+				)
+			)
+		)
+		(property "Footprint" ""
+			(at 107.95 200.66 0)
+			(effects
+				(font
+					(size 1.27 1.27)
+				)
+				(hide yes)
+			)
+		)
+		(property "Datasheet" ""
+			(at 107.95 200.66 0)
+			(effects
+				(font
+					(size 1.27 1.27)
+				)
+				(hide yes)
+			)
+		)
+		(property "Description" "Power symbol creates a global label with name \"+5V\""
+			(at 107.95 200.66 0)
+			(effects
+				(font
+					(size 1.27 1.27)
+				)
+				(hide yes)
+			)
+		)
+		(pin "1"
+		)
+		(instances
+			(project "spigate"
+				(path "/67c76d3f-b195-4782-8b26-36a2c4e1ea55"
+					(reference "#PWR08")
+					(unit 1)
+				)
+			)
+		)
+	)
+	(symbol
 		(lib_id "Device:C_Small")
 		(at 351.79 196.85 0)
@@
 	(symbol
 		(lib_id "power:+5V")
-		(at 116.84 191.77 0)
+		(at 118.11 191.77 0)
 		(unit 1)
 		(exclude_from_sim no)
@@
 		(dnp no)
 		(property "Reference" "#PWR07"
-			(at 116.84 195.58 0)
+			(at 118.11 195.58 0)
 			(effects
 				(font
@@
 		)
 		(property "Value" "+5V"
-			(at 119.38 190.5 0)
+			(at 120.65 190.5 0)
 			(effects
 				(font
@@
 		)
 		(property "Footprint" ""
-			(at 116.84 191.77 0)
+			(at 118.11 191.77 0)
 			(effects
 				(font
@@
 		)
 		(property "Datasheet" ""
-			(at 116.84 191.77 0)
+			(at 118.11 191.77 0)
 			(effects
 				(font
@@
 		)
 		(property "Description" "Power symbol creates a global label with name \"+5V\""
-			(at 116.84 191.77 0)
+			(at 118.11 191.77 0)
 			(effects
 				(font
@@
 	(symbol
 		(lib_id "Device:LED")
-		(at 116.84 203.2 90)
+		(at 118.11 203.2 90)
 		(unit 1)
 		(exclude_from_sim no)
@@
 		(fields_autoplaced yes)
 		(property "Reference" "D1"
-			(at 120.65 203.5174 90)
+			(at 121.92 203.5174 90)
 			(effects
 				(font
@@
 		)
 		(property "Value" "LED"
-			(at 120.65 206.0574 90)
+			(at 121.92 206.0574 90)
 			(effects
 				(font
@@
 		)
 		(property "Footprint" "LED_SMD:LED_0805_2012Metric_Pad1.15x1.40mm_HandSolder"
-			(at 116.84 203.2 0)
+			(at 118.11 203.2 0)
 			(effects
 				(font
@@
 		)
 		(property "Datasheet" "~"
-			(at 116.84 203.2 0)
+			(at 118.11 203.2 0)
 			(effects
 				(font
@@
 		)
 		(property "Description" "Light emitting diode"
-			(at 116.84 203.2 0)
+			(at 118.11 203.2 0)
 			(effects
 				(font
